Commit message: fixe front right leg

File: urdf/dream_walker.urdf (robot description, URDF)
Before this commit: robot dream_walker, 18 links, 17 joints
Links:
- added link A4_Link
Joints:
- added joint A4_joint: type fixed, parent A3_Link, child A4_Link, origin xyz=0 0 -0.44 rpy=0 0 0
- joint A0_joint: axis 0 0 0 -> (none); origin xyz=0.3 -0.083 0.55565 rpy=-1.57079632679 0 -1.57079632679 -> xyz=0.3485 -0.083 0 rpy=0 0 0
- joint A1_joint: axis 0 1 0 -> 1 0 0; limit lower=-9.42 upper=9.42 effort=1000 velocity=1000 -> lower=-3.1416 upper=3.1416 effort=25 velocity=1.5; origin xyz=0 0 0 rpy=-1.57079632679 0.07854 -1.57079632679 -> xyz=0.11 0 0 rpy=0 0 0
- joint A2_joint: axis 0 0 1 -> 0 1 0; limit lower=-9.42 upper=9.42 effort=1000 velocity=1000 -> lower=-3.1416 upper=3.1416 effort=25 velocity=1.5; origin xyz=-0.0065513 -0.083243 0.0315 rpy=0 0 -2.4347 -> xyz=0 -0.203 0 rpy=0 0 0
- joint A3_joint: axis 0 0 1 -> 0 1 0; origin xyz=0 -0.32 0.135 rpy=0 0 1.57079632679 -> xyz=0 -0.075 -0.32 rpy=0 0 0

Commit message: working urdf

File: urdf/dream_walker.urdf (robot description, URDF)
Before this commit: robot dream_walker, 19 links, 18 joints
Links:
- added link B4_Link
- added link C4_Link
- added link D4_Link
- link base_link: mass 1.5634 -> None
- link dummy: mass None -> 1.5634
Joints:
- added joint B4_joint: type fixed, parent B3_Link, child B4_Link, origin xyz=0 0 -0.44 rpy=0 0 0
- added joint C4_joint: type fixed, parent C3_Link, child C4_Link, origin xyz=0 0 -0.44 rpy=0 0 0
- added joint D4_joint: type fixed, parent D3_Link, child D4_Link, origin xyz=0 0 -0.44 rpy=0 0 0
- joint A1_joint: limit lower=-3.1416 upper=3.1416 effort=25 velocity=1.5 -> lower=-9.42 upper=9.42 effort=1000 velocity=1000
- joint A2_joint: limit lower=-3.1416 upper=3.1416 effort=25 velocity=1.5 -> lower=-9.42 upper=9.42 effort=1000 velocity=1000
- joint B0_joint: origin xyz=0.3 0.083 0.55565 rpy=-1.57079632679 0 -1.57079632679 -> xyz=0.3485 0.083 0 rpy=0 0 0
- joint B1_joint: axis 0 1 0 -> 1 0 0; origin xyz=0 0 0 rpy=-1.57079632679 0.07854 1.57079632679 -> xyz=0.11 0 0 rpy=0 0 0
- joint B2_joint: axis 0 0 1 -> 0 1 0; origin xyz=-0.0065513 -0.083243 0.0315 rpy=0 0 2.2777 -> xyz=0 0.203 0 rpy=0 0 0
- joint B3_joint: axis 0 0 1 -> 0 1 0; origin xyz=0 -0.32 0.135 rpy=0 0 -1.57079632679 -> xyz=0 0.075 -0.32 rpy=0 0 0
- joint C0_joint: origin xyz=-0.3 -0.083 0.55565 rpy=1.57079632679 0 -1.57079632679 -> xyz=-0.3485 -0.083 0 rpy=0 0 0
- joint C1_joint: axis 0 1 0 -> 1 0 0; origin xyz=0 0 0 rpy=-1.57079632679 0.07854 -1.57079632679 -> xyz=-0.11 0 0 rpy=0 0 0
- joint C2_joint: axis 0 0 1 -> 0 1 0; origin xyz=-0.0065513 -0.083243 0.0315 rpy=0 0 0.70686 -> xyz=0 -0.203 0 rpy=0 0 0
- joint C3_joint: axis 0 0 1 -> 0 1 0; origin xyz=0 -0.32 0.135 rpy=0 0 1.57079632679 -> xyz=0 -0.075 -0.32 rpy=0 0 0
- joint D0_joint: origin xyz=-0.3 0.083 0.55565 rpy=1.57079632679 0 -1.57079632679 -> xyz=-0.3485 0.083 0 rpy=0 0 0
- joint D1_joint: axis 0 1 0 -> 1 0 0; origin xyz=0 0 0 rpy=-1.57079632679 0.07854 1.57079632679 -> xyz=-0.11 0 0 rpy=0 0 0
- joint D2_joint: axis 0 0 1 -> 0 1 0; origin xyz=-0.0065513 -0.083243 0.0315 rpy=0 0 -0.86394 -> xyz=0 0.203 0 rpy=0 0 0
- joint D3_joint: axis 0 0 1 -> 0 1 0; origin xyz=0 -0.32 0.135 rpy=0 0 -1.57079632679 -> xyz=0 0.075 -0.32 rpy=0 0 0
- joint dummy_joint: child base_link -> dummy; parent dummy -> base_link
